File: PCB/PCB/PCB.kicad_pcb (KiCad board)
At the start: 4 copper layers, 83.1 x 50.9 mm, 53 parts, among them J1 AudioJack Right, J2 USB_B_Micro, J3 AudioJack Left, J4 6PIN DISPLAY CONNECTOR, J5 CONN BAT, Q1 BC817, Q2 BC817, Q3 BSS84, U1 ESP32-S3-WROOM-1, U2 CP2102N-Axx-xQFN28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

Commit message: Removed Errors
Routing:
- net VBUS: track 31.1 -> 29.8 mm
- net Net-(Q1-E): track 4.15 -> 4.71 mm

Commit message: Removed Errors
Parts:
- J1: value AudioJack Right -> Pre Right
- J3: value AudioJack Left -> Pre Left
Other:
- board text removed: "PWR LED"
Changed lines of the file:
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@@
     (property "ki_keywords" "LED diode")
     (attr smd)
-    (fp_text reference "D6" (at 0 -1.65) (layer "F.SilkS")
+    (fp_text reference "D6" (at -0.75 4.1) (layer "F.SilkS")
         (effects (font (size 1 1) (thickness 0.15)))
     )
-    (fp_text value "PWR_LED" (at 0 1.65) (layer "F.Fab")
+    (fp_text value "PWR_LED" (at 1.6 2.75) (layer "F.Fab")
         (effects (font (size 1 1) (thickness 0.15)))
     )
@@
     (property "ki_keywords" "cap capacitor")
     (attr smd)
-    (fp_text reference "C14" (at 0 -1.68 90) (layer "F.SilkS")
+    (fp_text reference "C14" (at -2.9 -0.2 90) (layer "F.SilkS")
         (effects (font (size 1 1) (thickness 0.15)))
     )
-    (fp_text value "100nF" (at 0 1.68 90) (layer "F.Fab")
+    (fp_text value "100nF" (at -2.15 -1.5 -90) (layer "F.Fab")
         (effects (font (size 1 1) (thickness 0.15)))
     )
@@
     (property "ki_keywords" "R res resistor")
     (attr smd)
-    (fp_text reference "R9" (at 0 -1.65) (layer "F.SilkS")
+    (fp_text reference "R9" (at -1.85 1.65) (layer "F.SilkS")
         (effects (font (size 1 1) (thickness 0.15)))
     )
@@
         (effects (font (size 1 1) (thickness 0.15)))
     )
-    (fp_text value "10µF" (at 0 1.68) (layer "F.Fab")
+    (fp_text value "10µF" (at 3.71225 0.04225) (layer "F.Fab")
         (effects (font (size 1 1) (thickness 0.15)))
     )
@@
         (effects (font (size 1 1) (thickness 0.15)))
     )
-    (fp_text value "AudioJack Right" (at 0 -10) (layer "F.Fab")
+    (fp_text value "Pre Right" (at -1.7 7.3) (layer "F.Fab")
         (effects (font (size 1 1) (thickness 0.15)))
     )
@@
         (effects (font (size 1 1) (thickness 0.15)))
     )
-    (fp_text value "CONN BAT" (at 0 4.87 90) (layer "F.Fab")
+    (fp_text value "CONN BAT" (at 2.50775 -0.86275 180) (layer "F.Fab")
         (effects (font (size 1 1) (thickness 0.15)))
     )
@@
     (property "ki_keywords" "R res resistor")
     (attr smd)
-    (fp_text reference "R12" (at 0 -1.65) (layer "F.SilkS")
+    (fp_text reference "R12" (at 0.85 -1.65) (layer "F.SilkS")
         (effects (font (size 1 1) (thickness 0.15)))
     )
@@
     (property "ki_keywords" "audio dac 2ch 24bit 96kHz")
     (attr smd)
-    (fp_text reference "U4" (at 0 -3.65) (layer "F.SilkS")
+    (fp_text reference "U4" (at -1.65 -4.9) (layer "F.SilkS")
         (effects (font (size 1 1) (thickness 0.15)))
     )
-    (fp_text value "UDA1334ATS" (at 0 3.65) (layer "F.Fab")
+    (fp_text value "UDA1334ATS" (at -1.75 -3.65) (layer "F.Fab")
         (effects (font (size 1 1) (thickness 0.15)))
     )
@@
         (effects (font (size 1 1) (thickness 0.15)))
     )
-    (fp_text value "Speaker Left" (at 2.78 7.75) (layer "F.Fab")
+    (fp_text value "Speaker Left" (at 1.565 7.15) (layer "F.Fab")
         (effects (font (size 1 1) (thickness 0.15)))
     )
@@
         (effects (font (size 1 1) (thickness 0.15)))
     )
-    (fp_text value "47µF" (at 0 5.2 90) (layer "F.Fab")
+    (fp_text value "47µF" (at -0.1 -6.6 90) (layer "F.Fab")
         (effects (font (size 1 1) (thickness 0.15)))
     )
@@
     (property "ki_keywords" "R res resistor")
     (attr smd)
-    (fp_text reference "R16" (at 0 -1.65) (layer "F.SilkS")
+    (fp_text reference "R16" (at 3.95 -0.3) (layer "F.SilkS")
         (effects (font (size 1 1) (thickness 0.15)))
     )
-    (fp_text value "10K" (at 0 1.65) (layer "F.Fab")
+    (fp_text value "10K" (at 3.95 1.05) (layer "F.Fab")
         (effects (font (size 1 1) (thickness 0.15)))
     )
@@
         (effects (font (size 1 1) (thickness 0.15)))
     )
-    (fp_text value "Speaker Right" (at 2.78 7.75) (layer "F.Fab")
+    (fp_text value "Speaker Right" (at 3.015 6.75) (layer "F.Fab")
         (effects (font (size 1 1) (thickness 0.15)))
     )
@@
     (property "ki_keywords" "cap capacitor")
     (attr smd)
-    (fp_text reference "C7" (at 0 -1.68 90) (layer "F.SilkS")
+    (fp_text reference "C7" (at 1.05 -2.15 90) (layer "F.SilkS")
         (effects (font (size 1 1) (thickness 0.15)))
     )
-    (fp_text value "10µF" (at 0 1.68 90) (layer "F.Fab")
+    (fp_text value "10µF" (at 0 2.65 90) (layer "F.Fab")
         (effects (font (size 1 1) (thickness 0.15)))
     )
@@
         (effects (font (size 1 1) (thickness 0.15)))
     )
-    (fp_text value "MCP73831-3-OT" (at 0 2.4) (layer "F.Fab")
+    (fp_text value "MCP73831-3-OT" (at 0 3.09225) (layer "F.Fab")
         (effects (font (size 1 1) (thickness 0.15)))
     )
@@
         (effects (font (size 1 1) (thickness 0.15)))
     )
-    (fp_text value "AudioJack Left" (at 0 -10) (layer "F.Fab")
+    (fp_text value "Pre Left" (at 0.05 7.3) (layer "F.Fab")
         (effects (font (size 1 1) (thickness 0.15)))
     )
@@
   (gr_rect (start 76.92 30.48) (end 160.02 81.35)
     (stroke (width 0.1) (type default)) (fill none) (layer "Edge.Cuts"))
-  (gr_text "PWR LED" (at 78.3 34) (layer "F.SilkS")
-    (effects (font (size 1 1) (thickness 0.25) bold) (justify left bottom))
-  )
   (gr_text "Felix Strauß\nVersion 1.0" (at 159.7 80.9) (layer "F.SilkS")
     (effects (font (size 1.5 1.5) (thickness 0.3) bold) (justify right bottom))
