File: PCB/PCB/PCB.kicad_pcb (KiCad board)
At the start: 4 copper layers, 83.1 x 50.9 mm, 53 parts, among them J1 Pre Right, J2 USB_B_Micro, J3 Pre Left, J4 6PIN DISPLAY CONNECTOR, J5 CONN BAT, Q1 BC817, Q2 BC817, Q3 BSS84, U1 ESP32-S3-WROOM-1, U2 CP2102N-Axx-xQFN28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

Commit message: Removed Errors
Parts:
- LS L: renamed from LS1
- LS R: renamed from LS2
- moved D1 5.16 mm to (86.4, 65.7), turned to 90 degrees
- moved D2 5.06 mm to (88.8, 65.2), turned to 90 degrees
- moved D3 4.50 mm to (86.4, 69.0)
- moved J2 3.39 mm to (80.6, 67.2)
- moved J1 3.17 mm to (130.4, 35.4), turned to 180 degrees
- moved J3 3.05 mm to (117.2, 35.5), turned to 180 degrees
- moved R2 2.12 mm to (92.1, 69.0)
- moved C2 0.79 mm to (100.6, 71.4)
- moved R1 0.79 mm to (94.5, 74.2)
- moved R3 0.79 mm to (97.1, 71.4)
- moved C1 0.79 mm to (96.5, 74.2)
- moved R15 0.71 mm to (107.4, 44.2)
- moved C16 0.71 mm to (107.4, 46.3)
- moved D5 0.65 mm to (100.8, 40.9)
- moved R14 0.65 mm to (103.5, 40.0)
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Routing:
- net Net-(U5-INL): track 47.0 -> 54.4 mm
- net GND: track 109.8 -> 103.3 mm, vias 24 -> 23
- net Net-(U5-INR): track 21.1 -> 25.7 mm
- net Net-(U2-VBUS): track 6.28 -> 8.93 mm
- net Net-(D3-A1): track 9.08 -> 11.1 mm, vias 0 -> 2
- net VBUS: track 29.8 -> 31.2 mm
- net Net-(D2-A1): track 12.0 -> 13.1 mm
- net Net-(U2-~{RST}): track 1.90 -> 2.72 mm
- net Net-(U6-PROG): track 1.87 -> 2.55 mm
- net Net-(D1-A1): track 13.2 -> 12.6 mm, vias 2 -> 0
- net Net-(D5-K): track 2.11 -> 2.73 mm
Other:
- board text added: "BAT + -"
- board text added: "CHG_LED"
- board text added: "PWR_LED"

Commit message: PCB finished
Parts:
- J1: value Pre Right -> AudioJack Right
- J2: value USB_B_Micro -> USB_C_Receptacle_USB2.0; footprint Connector_USB:USB_Micro-B_Molex-105017-0001 -> Connector_USB:USB_C_Receptacle_GCT_USB4105-xx-A_16P_TopMnt_Horizontal
- J3: value Pre Left -> AudioJack Left
- LS1: renamed from LS L
- LS2: renamed from LS R
- moved C15 5.80 mm to (144.6, 69.1), turned to 0 degrees
- moved C11 3.72 mm to (153.8, 59.7), turned to -90 degrees
- moved R11 3.19 mm to (151.8, 59.7)
- moved C1 3.07 mm to (94.0, 75.9)
- moved R1 3.07 mm to (92.0, 75.9)
- moved C14 3.04 mm to (138.4, 65.0)
- moved C7 2.98 mm to (132.8, 68.8)
- moved R9 2.98 mm to (132.2, 71.5)
- moved C8 2.71 mm to (156.6, 45.6)
- moved C9 2.65 mm to (156.6, 50.2)
- moved C2 2.01 mm to (100.6, 73.4)
- moved R3 2.01 mm to (97.1, 73.4)
- moved C17 1.91 mm to (134.9, 51.8)
- moved R12 1.91 mm to (131.8, 46.2)
- moved C12 1.91 mm to (140.8, 47.0)
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Routing:
- net GND: track 103.3 -> 97.9 mm, vias 23 -> 24
- net Net-(U4-Vref(DAC)): track 6.52 -> 11.0 mm
- net Net-(U5-INL): track 54.4 -> 57.8 mm
- net Net-(U2-VBUS): track 8.93 -> 11.8 mm
- net Net-(U5-VREF): track 2.20 -> 4.85 mm
- net Net-(U5-VDD): track 15.1 -> 17.8 mm
- net /txd: track 30.2 -> 32.6 mm
- net Net-(D3-A1): track 11.1 -> 13.4 mm, vias 2 -> 0
- net /rxd: track 28.6 -> 30.8 mm
- net Net-(U2-~{RST}): track 2.72 -> 4.75 mm
- net Net-(D1-A1): track 12.6 -> 10.7 mm
- net Net-(Q2-E): track 4.11 -> 5.72 mm
- net Net-(Q1-E): track 4.71 -> 6.32 mm
- net Net-(U5-LOUT-): track 21.4 -> 19.9 mm, vias 0 -> 2
- net /GPIO0: track 33.4 -> 34.5 mm
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Other:
- board text added: "Version 1.0 ©Felix Strauß, 2023"
- board text added: "https://github.com/fstrs/PCB-Kurs"
- board text removed: "Felix Strauß Version 1.0"

Commit message: finished Documentation
Parts:
- D5: value LED -> CHG_LED
- R6, R7: value R -> 1K
Connections:
- J2 pad A7: unconnected-(J2-D--PadA7) -> Net-(D1-A1)
- J2 pad B6: unconnected-(J2-D+-PadB6) -> Net-(D2-A1)
- U2 pad 25: /rxd -> /txd
- U2 pad 26: /txd -> /rxd
Routing:
- net Net-(D1-A1): track 10.7 -> 13.5 mm
- net /txd: track 32.6 -> 30.5 mm
- net /rxd: track 30.8 -> 32.8 mm
- net Net-(D2-A1): track 12.0 -> 13.8 mm
- net /GPIO0: track 34.5 -> 33.7 mm
