File: PCB/PCB/PCB.kicad_sch (KiCad schematic)
At the start: 53 parts, among them J1 AudioJack Right, J2 USB_B_Micro, J3 AudioJack Left, J4 6PIN DISPLAY CONNECTOR, Q1 BC817, Q2 BC817, Q3 BSS84, U1 ESP32-S3-WROOM-1, U2 CP2102N-Axx-xQFN28, U3 NCP1117-3.3_SOT223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

Commit message: PCB Verion 1.0
Parts:
- removed C10, C13: 47µF, symbol Device:C
- removed C6: 100nF, symbol Device:C
- added C17, C18: 47µF, Capacitor_SMD:C_Elec_8x10.2, symbol Device:C_Polarized
- added J5: CONN BAT, Connector_PinHeader_2.54mm:PinHeader_1x02_P2.54mm_Vertical, symbol Connector:Conn_01x02_Socket
- C1, C11, C12, C14, C16, C2, C3, C4, C5, C8, C9: footprint (none) -> Capacitor_SMD:C_0805_2012Metric
- C15: footprint (none) -> Capacitor_SMD:C_Elec_8x10.2
- C7: value 47µF -> 10µF; footprint (none) -> Capacitor_SMD:C_0805_2012Metric
- D5, D6: footprint (none) -> LED_SMD:LED_0805_2012Metric
- J1: footprint Connector_Audio:Jack_XLR_Neutrik_NC3FAAH1-0_Horizontal -> Connector_Audio:Jack_3.5mm_CUI_SJ1-3523N_Horizontal
- J3: footprint (none) -> Connector_Audio:Jack_3.5mm_CUI_SJ1-3523N_Horizontal
- J4: footprint (none) -> Connector_PinHeader_2.54mm:PinHeader_1x06_P2.54mm_Vertical
- LS1, LS2: footprint (none) -> TerminalBlock:TerminalBlock_Altech_AK300-2_P5.00mm
- R1, R10, R11, R12, R13, R14, R15, R16, R2, R3, R4, R5, R6, R7, R8, R9: footprint (none) -> Resistor_SMD:R_0805_2012Metric
Connections:
- net +BATT: now also J5.1 (Pin_1)
- net GND: now also J5.2 (Pin_2)
- net at U4.16 (VOUTR): now also C17.1
- net at R12.2, R13.1: now also C17.2
- net at U4.14 (VOUTL): now also C18.1
- net at R10.1, R11.1: now also C18.2
- no-connect marks 28 -> 44

Commit message: PCB finished
Parts:
- removed J2: USB_B_Micro, Connector_USB:USB_Micro-B_Molex-105017-0001, symbol Connector:USB_B_Micro
- added J2: USB_C_Receptacle_USB2.0, Connector_USB:USB_C_Receptacle_GCT_USB4105-xx-A_16P_TopMnt_Horizontal, symbol Connector:USB_C_Receptacle_USB2.0
Connections:
- net GND: now also J2.A1 (GND), J2.A12 (GND), J2.B1 (GND), J2.B12 (GND), J2.S1 (SHIELD)
- net at D3.1 (A1), R2.2: now also J2.A4 (VBUS), J2.A9 (VBUS), J2.B4 (VBUS), J2.B9 (VBUS)
- net at D1.1 (A1), U2.5 (D-): now also J2.B7 (D-)
- net at D2.1 (A1), U2.4 (D+): now also J2.A6 (D+)
- no-connect marks 44 -> 49
Other:
- moved on the sheet: C1, C2, D1, D2, D3, D6, Q1, Q2, R1, R16, R2, R3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
